File: bnc_shield_pcb/bnc_shield.kicad_pcb (KiCad board)
At the start: 2 copper layers, 91.4 x 91.4 mm, 41 parts, among them J1 Conn_Coaxial, J10 Conn_Coaxial, J11 Conn_Coaxial, J12 Conn_01x06_Male, J13 Conn_01x10_Male, J14 Conn_01x08_Male, J2 Conn_Coaxial, J3 Conn_Coaxial, J4 Conn_Coaxial, J5 Conn_Coaxial, J6 Conn_01x07_Male, J7 Conn_Coaxial, J8 Conn_Coaxial, J9 Conn_Coaxial, P1 Power, P2 Analog, P3 Digital, P4 Digital, P5 CONN_01X01, P7 CONN_01X01, P8 CONN_01X01, SW1 SW_MEC_5E

Commit message: Version 2, as ordered
Parts:
- removed the REF** at (122.4, 94.6)
- removed the REF** at (132.6, 104.8)
- removed the REF** at (145.3, 113.7)
- removed the REF** at (163.1, 94.6)
- removed the REF** at (125.0, 113.7)
- removed the REF** at (152.9, 104.8)
- removed the REF** at (132.6, 94.6)
- removed the REF** at (163.1, 104.8)
- removed the REF** at (165.6, 113.7)
- removed the REF** at (135.1, 113.7)
- removed the REF** at (142.7, 104.8)
- removed the REF** at (142.7, 94.6)
- removed the REF** at (122.4, 104.8)
- removed the REF** at (155.4, 113.7)
- removed the REF** at (152.9, 94.6)
- added G***: LOGO, test:arduino_bnc_qr, F.Cu at (118.7, 101.6)
- added REF**: 8_by_8_prototype_area, prototyping:8_by_8_prototype_area, F.Cu at (135.9, 105.4)
- added REF**: 8_by_8_prototype_area, prototyping:8_by_8_prototype_area, F.Cu at (156.2, 105.4)
- 3 jump: footprint Jumper:SolderJumper-3_P1.3mm_Bridged12_Pad1.0x1.5mm -> Misc_custom:SolderJumper-3-P2.54mm_Bridged12
- A4 jump: footprint Jumper:SolderJumper-3_P1.3mm_Bridged12_Pad1.0x1.5mm -> Misc_custom:SolderJumper-3-P2.54mm_Bridged12
- SW1: footprint digikey-footprints:Switch_Tactile_SMD_6x6mm_PTS645 -> digikey-footprints:Switch_Tactile_THT_6x6mm
- moved 3 jump 3.72 mm to (177.8, 99.6)
- moved SW1 1.71 mm to (112.9, 74.2)
Routing:
- net /A4(SDA): track 19.1 -> 24.8 mm
- net Net-(J7-Pad1): track 10.2 -> 14.0 mm
- net /3(**): track 46.6 -> 49.9 mm
- net Net-(J5-Pad1): track 9.02 -> 12.2 mm
- net Net-(J16-Pad1): track 3.81 -> 5.27 mm
- net GND: track 23.0 -> 21.7 mm
- net Net-(J15-Pad1): track 5.17 -> 4.65 mm
Other:
- board text added: "V2, 07/17/23"
- board text added: "github.com/jazzlw/arduino_bnc"
- board text removed: "08/22/22"
