File: bnc_shield_pcb/bnc_shield.kicad_sch (KiCad schematic)
At the start: 26 parts, among them J1 Conn_Coaxial, J10 Conn_Coaxial, J11 Conn_Coaxial, J12 Conn_01x06_Male, J13 Conn_01x10_Male, J14 Conn_01x08_Male, J15 Conn_01x01_Male, J16 Conn_01x01_Male, J2 Conn_Coaxial, J3 Conn_Coaxial, J4 Conn_Coaxial, J5 Conn_Coaxial, J6 Conn_01x07_Male, J7 Conn_Coaxial, J8 Conn_Coaxial, J9 Conn_Coaxial, P1 Power, P2 Analog, P3 Digital, P4 Digital, P5 CONN_01X01, P7 CONN_01X01, P8 CONN_01X01, SW1 SW_MEC_5E

Commit message: Version 2, as ordered
Parts:
- JP1, JP2: footprint Jumper:SolderJumper-3_P1.3mm_Bridged12_Pad1.0x1.5mm -> Misc_custom:SolderJumper-3-P2.54mm_Bridged12
- SW1: footprint digikey-footprints:Switch_Tactile_SMD_6x6mm_PTS645 -> digikey-footprints:Switch_Tactile_THT_6x6mm
Changed lines of the file:
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@@
       (effects (font (size 1.27 1.27)) (justify left))
     )
-    (property "Footprint" "Jumper:SolderJumper-3_P1.3mm_Bridged12_Pad1.0x1.5mm" (id 2) (at 126.365 104.14 0)
+    (property "Footprint" "Misc_custom:SolderJumper-3-P2.54mm_Bridged12" (id 2) (at 126.365 104.14 0)
       (effects (font (size 1.27 1.27)) hide)
     )
@@
     (property "Reference" "SW1" (id 0) (at 255.27 94.0775 0))
     (property "Value" "SW_MEC_5E" (id 1) (at 255.27 96.8526 0))
-    (property "Footprint" "digikey-footprints:Switch_Tactile_SMD_6x6mm_PTS645" (id 2) (at 255.27 95.885 0)
+    (property "Footprint" "digikey-footprints:Switch_Tactile_THT_6x6mm" (id 2) (at 255.27 95.885 0)
       (effects (font (size 1.27 1.27)) hide)
     )
@@
       (effects (font (size 1.27 1.27)) (justify left))
     )
-    (property "Footprint" "Jumper:SolderJumper-3_P1.3mm_Bridged12_Pad1.0x1.5mm" (id 2) (at 167.64 45.72 0)
+    (property "Footprint" "Misc_custom:SolderJumper-3-P2.54mm_Bridged12" (id 2) (at 167.64 45.72 0)
       (effects (font (size 1.27 1.27)) hide)
     )
@@
     )
     (path "/053c8083-a9af-4404-9cbb-5f2f2c004e29"
-      (reference "JP1") (unit 1) (value "jumper") (footprint "Jumper:SolderJumper-3_P1.3mm_Bridged12_Pad1.0x1.5mm")
+      (reference "JP1") (unit 1) (value "jumper") (footprint "Misc_custom:SolderJumper-3-P2.54mm_Bridged12")
     )
     (path "/a4c5c756-5c56-44ed-8cdc-4543d4cb82ab"
-      (reference "JP2") (unit 1) (value "jumper") (footprint "Jumper:SolderJumper-3_P1.3mm_Bridged12_Pad1.0x1.5mm")
+      (reference "JP2") (unit 1) (value "jumper") (footprint "Misc_custom:SolderJumper-3-P2.54mm_Bridged12")
     )
     (path "/00000000-0000-0000-0000-000056d70129"
@@
     )
     (path "/669281f0-5788-4ca9-ae77-1c6b3ce2c43a"
-      (reference "SW1") (unit 1) (value "SW_MEC_5E") (footprint "digikey-footprints:Switch_Tactile_SMD_6x6mm_PTS645")
-    )
-  )
+      (reference "SW1") (unit 1) (value "SW_MEC_5E") (footprint "digikey-footprints:Switch_Tactile_THT_6x6mm")
+    )
+  )
